Commit message: documentation added, camera inverted

File: install/dobot_rviz/share/dobot_rviz/urdf/cr5_robot.urdf (robot description, URDF)
Before this commit: robot cr5_robot, 9 links, 8 joints
Links:
- link zed: geometry collision box size=0.18 0.18 0.05; visual box size=0.18 0.18 0.05

Commit message: camera position modified, dobot_stop.sh modified

File: install/dobot_rviz/share/dobot_rviz/urdf/cr5_robot.urdf (robot description, URDF)
Before this commit: robot cr5_robot, 9 links, 8 joints
Links:
- link zed: geometry collision box size=0.12 0.10 0.05; visual box size=0.12 0.12 0.05

Commit message: zed dimentions in urdf changed, dobot_startup modified (now reworked_map is correctly launched)

File: install/dobot_rviz/share/dobot_rviz/urdf/cr5_robot.urdf (robot description, URDF)
Before this commit: robot cr5_robot, 9 links, 8 joints
Links:
- link zed: geometry collision box size=0.18 0.25 0.05; visual box size=0.22 0.25 0.05
